Commit message: fix broken joints

File: baby_yeti_description/urdf/baby_yeti.urdf (robot description, URDF)
Before this commit: robot lawnbot, 6 links, 5 joints
Links:
- link base_link: mass None -> 45
Joints:
- joint base_to_wheel_bl: origin xyz=0.3 -0.2375 -0.1 rpy=1.57 -3.14159 0 -> xyz=-0.3 0.2375 -0.1 rpy=1.57 0 0
- joint base_to_wheel_br: origin xyz=0.3 0.2375 -0.1 rpy=1.57 -3.14159 0 -> xyz=-0.3 -0.2375 -0.1 rpy=1.57 0 0
- joint base_to_wheel_fl: origin xyz=-0.3 -0.2375 -0.1 rpy=1.57 -3.14159 0 -> xyz=0.3 0.2375 -0.1 rpy=1.57 0 0
- joint base_to_wheel_fr: origin xyz=-0.3 0.2375 -0.1 rpy=1.57 -3.14159 0 -> xyz=0.3 -0.2375 -0.1 rpy=1.57 0 0
